File: keyboard.kicad_pcb (KiCad board)
At the start: 2 copper layers, 203.4 x 107.7 mm, 50 parts, among them J1 TRRS, SW00 Key, SW01 Key, SW02 Key, SW03 Key, SW10 Key, SW11 Key, SW12 Key, SW13 Key, SW14 Key, SW15 Key, SW16 Key, SW17 Key, SW18 Key, SW20 Key, SW21 Key, SW22 Key, SW23 Key, SW24 Key, SW25 Key, SW26 Key, SW27 Key, SW28 Key, SW30 Key, SW31 Key, SW32 Key, SW33 Key, SW34 Key, SW35 Key, SW36 Key, SW37 Key, SW38 Key, SW40 Key, SW41 Key, SW42 Key, SW43 Key, SW44 Key, SW45 Key, SW46 Key, SW47 Key, SW48 Key, U1 ProMicro

Commit message: remove area under palm
Routing:
- net row4: track 209.2 -> 235.4 mm
Other:
- outline, holes or cut-outs redrawn
Changed lines of the file:
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@@
   (gr_line (start 185.933943 84.58049) (end 183.345753 94.239748)
     (stroke (width 0.12) (type solid)) (layer "Edge.Cuts"))
+  (gr_arc (start 139.000764 116.780478) (mid 138.393558 116.314552) (end 138.293657 115.555733)
+    (stroke (width 0.12) (type solid)) (layer "Edge.Cuts"))
   (gr_line (start 76.78 48) (end 70.78 48)
     (stroke (width 0.12) (type solid)) (layer "Edge.Cuts"))
@@
   (gr_line (start 232.830502 136.777818) (end 179.650884 127.400816)
     (stroke (width 0.12) (type solid)) (layer "Edge.Cuts"))
-  (gr_arc (start 117.519499 112.23964) (mid 117.942117 111.507644) (end 118.774513 111.36087)
-    (stroke (width 0.12) (type solid)) (layer "Edge.Cuts"))
   (gr_arc (start 100.768166 50.017579) (mid 104.875885 50.099138) (end 108.981748 50.247128)
     (stroke (width 0.12) (type solid)) (layer "Edge.Cuts"))
@@
   (gr_arc (start 194.62096 59.887508) (mid 195.049586 59.302936) (end 195.760534 59.161519)
     (stroke (width 0.12) (type solid)) (layer "Edge.Cuts"))
-  (gr_line (start 117.519499 112.23964) (end 116.788826 120.591269)
+  (gr_line (start 118.147883 105.05718) (end 116.788826 120.591269)
     (stroke (width 0.12) (type solid)) (layer "Edge.Cuts"))
   (gr_line (start 117.463578 44.594125) (end 109.494021 43.896879)
@@
   (gr_arc (start 139.264846 51.383681) (mid 140.089577 52.532513) (end 138.940745 53.357246)
     (stroke (width 0.12) (type solid)) (layer "Edge.Cuts"))
+  (gr_arc (start 139.397025 107.237461) (mid 140.066769 107.684969) (end 140.189303 108.481088)
+    (stroke (width 0.12) (type solid)) (layer "Edge.Cuts"))
   (gr_arc (start 132.963412 50.429249) (mid 132.318785 50.061938) (end 132.104654 49.351579)
     (stroke (width 0.12) (type solid)) (layer "Edge.Cuts"))
   (gr_arc (start 117.463578 44.594125) (mid 118.372618 45.677475) (end 117.289267 46.586515)
     (stroke (width 0.12) (type solid)) (layer "Edge.Cuts"))
+  (gr_arc (start 118.147883 105.05718) (mid 118.508889 104.371979) (end 119.250898 104.150059)
+    (stroke (width 0.12) (type solid)) (layer "Edge.Cuts"))
   (gr_line (start 174.998839 125.390856) (end 176.422345 120.078257)
     (stroke (width 0.12) (type solid)) (layer "Edge.Cuts"))
@@
   (gr_line (start 153.339152 55.878224) (end 144.84099 54.379769)
     (stroke (width 0.12) (type solid)) (layer "Edge.Cuts"))
-  (gr_line (start 173.774094 126.097963) (end 118.774513 111.36087)
+  (gr_line (start 173.774094 126.097963) (end 139.000764 116.780478)
     (stroke (width 0.12) (type solid)) (layer "Edge.Cuts"))
   (gr_arc (start 110.022044 49.335256) (mid 109.685014 50.000099) (end 108.981748 50.247126)
@@
   (gr_arc (start 123.266435 47.109449) (mid 122.357397 46.026099) (end 123.440746 45.117061)
     (stroke (width 0.12) (type solid)) (layer "Edge.Cuts"))
+  (gr_arc (start 119.250898 104.150057) (mid 125.98312 104.988487) (end 132.683213 106.053635)
+    (stroke (width 0.12) (type solid)) (layer "Edge.Cuts"))
   (gr_arc (start 189.677529 78.336648) (mid 188.452784 79.043755) (end 187.745677 77.819009)
     (stroke (width 0.12) (type solid)) (layer "Edge.Cuts"))
+  (gr_line (start 139.397025 107.237462) (end 132.683213 106.053635)
+    (stroke (width 0.12) (type solid)) (layer "Edge.Cuts"))
   (gr_arc (start 179.650884 127.400815) (mid 178.686906 127.223771) (end 177.72554 127.033053)
     (stroke (width 0.12) (type solid)) (layer "Edge.Cuts"))
@@
     (stroke (width 0.12) (type solid)) (layer "Edge.Cuts"))
   (gr_arc (start 76.78 48) (mid 77.78 49) (end 76.78 50)
+    (stroke (width 0.12) (type solid)) (layer "Edge.Cuts"))
+  (gr_line (start 138.293657 115.555733) (end 140.189303 108.481088)
     (stroke (width 0.12) (type solid)) (layer "Edge.Cuts"))
   (gr_arc (start 152.255589 52.640883) (mid 151.844358 53.286387) (end 151.097133 53.452043)
@@
   (segment (start 67.51 97.952526) (end 67.51 82.75) (width 0.25) (layer "F.Cu") (net 4))
   (segment (start 68.5 98.942526) (end 67.51 97.952526) (width 0.25) (layer "F.Cu") (net 4))
-  (segment (start 147 110.5) (end 117 110.5) (width 0.25) (layer "B.Cu") (net 4))
   (segment (start 169.711722 118.559683) (end 181.559683 118.559683) (width 0.25) (layer "B.Cu") (net 4))
-  (segment (start 110.395812 114.781975) (end 91.190176 114.781975) (width 0.25) (layer "B.Cu") (net 4))
   (segment (start 186.370948 123.370948) (end 192.673506 123.370948) (width 0.25) (layer "B.Cu") (net 4))
   (segment (start 204.370948 123.370948) (end 207.496615 126.496615) (width 0.25) (layer "B.Cu") (net 4))
+  (segment (start 143 107.5) (end 137 101.5) (width 0.25) (layer "B.Cu") (net 4))
   (segment (start 159.900941 113.900941) (end 164.559683 118.559683) (width 0.25) (layer "B.Cu") (net 4))
+  (segment (start 143 109.5) (end 143 107.5) (width 0.25) (layer "B.Cu") (net 4))
   (segment (start 207.496615 126.496615) (end 210.400046 126.496615) (width 0.25) (layer "B.Cu") (net 4))
-  (segment (start 112.718025 114.781975) (end 110.395812 114.781975) (width 0.25) (layer "B.Cu") (net 4))
-  (segment (start 150.400941 113.900941) (end 147 110.5) (width 0.25) (layer "B.Cu") (net 4))
   (segment (start 65.415225 104.396637) (end 70.717383 104.396637) (width 0.25) (layer "B.Cu") (net 4))
   (segment (start 192.673506 123.370948) (end 204.370948 123.370948) (width 0.25) (layer "B.Cu") (net 4))
   (segment (start 77.598656 114.804949) (end 72.599736 119.803869) (width 0.25) (layer "B.Cu") (net 4))
+  (segment (start 137 101.5) (end 102.5 101.5) (width 0.25) (layer "B.Cu") (net 4))
   (segment (start 222.496615 126.496615) (end 225.622282 129.622282) (width 0.25) (layer "B.Cu") (net 4))
+  (segment (start 110.395812 114.781975) (end 98 114.781975) (width 0.25) (layer "B.Cu") (net 4))
   (segment (start 70.717383 104.396637) (end 77.598656 111.27791) (width 0.25) (layer "B.Cu") (net 4))
-  (segment (start 152.325058 113.900941) (end 150.400941 113.900941) (width 0.25) (layer "B.Cu") (net 4))
+  (segment (start 98 106) (end 98 114.781975) (width 0.25) (layer "B.Cu") (net 4))
   (segment (start 210.400046 126.496615) (end 222.496615 126.496615) (width 0.25) (layer "B.Cu") (net 4))
   (segment (start 91.167202 114.804949) (end 77.598656 114.804949) (width 0.25) (layer "B.Cu") (net 4))
   (segment (start 91.190176 114.781975) (end 91.167202 114.804949) (width 0.25) (layer "B.Cu") (net 4))
+  (segment (start 147.400941 113.900941) (end 143 109.5) (width 0.25) (layer "B.Cu") (net 4))
   (segment (start 164.559683 118.559683) (end 169.711722 118.559683) (width 0.25) (layer "B.Cu") (net 4))
+  (segment (start 102.5 101.5) (end 98 106) (width 0.25) (layer "B.Cu") (net 4))
+  (segment (start 98 114.781975) (end 91.190176 114.781975) (width 0.25) (layer "B.Cu") (net 4))
   (segment (start 152.325058 113.900941) (end 159.900941 113.900941) (width 0.25) (layer "B.Cu") (net 4))
   (segment (start 77.598656 111.27791) (end 77.598656 114.804949) (width 0.25) (layer "B.Cu") (net 4))
   (segment (start 225.622282 129.622282) (end 228.126585 129.622282) (width 0.25) (layer "B.Cu") (net 4))
   (segment (start 181.559683 118.559683) (end 186.370948 123.370948) (width 0.25) (layer "B.Cu") (net 4))
-  (segment (start 117 110.5) (end 112.718025 114.781975) (width 0.25) (layer "B.Cu") (net 4))
+  (segment (start 152.325058 113.900941) (end 147.400941 113.900941) (width 0.25) (layer "B.Cu") (net 4))
   (segment (start 61.16 69.796) (end 61.16 66.24) (width 0.25) (layer "F.Cu") (net 5))
   (segment (start 61.16 66.24) (end 52.27 57.35) (width 0.25) (layer "F.Cu") (net 5))

Commit message: improve traces
Parts:
- moved R2 1.27 mm to (63.7, 79.2)
- moved R1 0.76 mm to (63.7, 76.7)
Routing:
- net col4: track 196.2 -> 208.0 mm
- net col6: track 233.5 -> 222.2 mm, vias 7 -> 5
- net col7: track 233.1 -> 241.1 mm, vias 7 -> 6
- net col2: track 195.5 -> 192.4 mm
- net row1: track 213.4 -> 211.0 mm
- net row2: track 186.6 -> 188.2 mm
- net row4: track 235.4 -> 236.8 mm
- net SCL: track 21.6 -> 20.3 mm
- net col1: track 171.9 -> 170.8 mm
- net row3: track 191.7 -> 190.8 mm
- net col3: track 212.3 -> 211.4 mm
- net col5: track 209.1 -> 209.9 mm, vias 5 -> 4
- net VCC: track 25.1 -> 24.3 mm
- net SDA: track 27.5 -> 26.7 mm
- net col8: track 254.3 -> 254.1 mm, vias 7 -> 6
